File: kicad/Vocab.sch (KiCad schematic (older format))
At the start: 40 parts, among them K1 CONN_3, K2 CONN_3, K3 CONN_3, K4 CONN_3, M1 Arduino, P1 CONN_1, P2 CONN_1, P4 CONN_1, P5 CONN_1, P6 CONN_2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

Commit message: Added manufacturer part numbers (except for Rs - generic 0805) Added stacking connectors to bom manually
Parts:
- C1, C2: MFN (none) -> MC1210B104K201CT; MFP (none) -> Multicomp
- C3, C4: MFN (none) -> AVES106M35C12T-F; MFP (none) -> Dubilier
- D1, D2, D3, D4: value 1n914 -> 1n4148; MFN (none) -> 1n4148W; MFP (none) -> Vishay
- K1, K2: MFN (none) -> 640457-2; MFP (none) -> TE Connectivity
- K3, K4: value CONN_3 -> NF
- L1, L2: MFN (none) -> 2512061217Y5; MFP (none) -> Fair-rite
- P1, P2, P4, P5: value CONN_1 -> NF
- P6: MFN (none) -> 640455-2; MFP (none) -> TE Connectivity
- U1: MFN (none) -> ADS1115IDGST; MFP (none) -> TI
- U2: MFN (none) -> 11aa02e48-I/TT; MFP (none) -> Microchip
Changed lines of the file:
@@
 F 2 "Socket_Strips:Socket_Strip_Straight_1x03" H 1650 3200 60  0001 C CNN
 F 3 "" H 1650 3200 60  0000 C CNN
+F 4 "640457-2" H 1650 3200 60  0001 C CNN "MFN"
+F 5 "TE Connectivity" H 1650 3200 60  0001 C CNN "MFP"
 	1    1650 3200
 	-1   0    0    -1
@@
 F 2 "Socket_Strips:Socket_Strip_Straight_1x03" H 1650 3900 60  0001 C CNN
 F 3 "" H 1650 3900 60  0000 C CNN
+F 4 "640457-2" H 1650 3900 60  0001 C CNN "MFN"
+F 5 "TE Connectivity" H 1650 3900 60  0001 C CNN "MFP"
 	1    1650 3900
 	-1   0    0    -1
@@
 F 2 "Capacitors_SMD:C_1210" H 4200 4300 60  0001 C CNN
 F 3 "" H 4200 4300 60  0000 C CNN
+F 4 "MC1210B104K201CT" H 4200 4300 60  0001 C CNN "MFN"
+F 5 "Multicomp" H 4200 4300 60  0001 C CNN "MFP"
 	1    4200 4300
 	0    -1   -1   0
@@
 F 2 "Capacitors_SMD:C_1210" H 3200 4300 60  0001 C CNN
 F 3 "" H 3200 4300 60  0000 C CNN
+F 4 "MC1210B104K201CT" H 3200 4300 60  0001 C CNN "MFN"
+F 5 "Multicomp" H 3200 4300 60  0001 C CNN "MFP"
 	1    3200 4300
 	0    -1   -1   0
@@
 L DIODE D1
 U 1 1 5468B880
-P 3200 4600
-F 0 "D1" H 3200 4700 40  0000 C CNN
-F 1 "1n914" H 3200 4500 40  0000 C CNN
-F 2 "Diodes_SMD:SOD-123" H 3200 4600 60  0001 C CNN
-F 3 "" H 3200 4600 60  0000 C CNN
-	1    3200 4600
+P 3205 4600
+F 0 "D1" H 3205 4700 40  0000 C CNN
+F 1 "1n4148" H 3205 4500 40  0000 C CNN
+F 2 "Diodes_SMD:SOD-123" H 3205 4600 60  0001 C CNN
+F 3 "" H 3205 4600 60  0000 C CNN
+F 4 "1n4148W" H 3205 4600 60  0001 C CNN "MFN"
+F 5 "Vishay" H 3205 4600 60  0001 C CNN "MFP"
+	1    3205 4600
 	1    0    0    -1
 $EndComp
@@
 P 3200 4900
 F 0 "D2" H 3200 5000 40  0000 C CNN
-F 1 "1n914" H 3200 4800 40  0000 C CNN
+F 1 "1n4148" H 3200 4800 40  0000 C CNN
 F 2 "Diodes_SMD:SOD-123" H 3200 4900 60  0001 C CNN
 F 3 "" H 3200 4900 60  0000 C CNN
+F 4 "1n4148W" H 3200 4900 60  0001 C CNN "MFN"
+F 5 "Vishay" H 3200 4900 60  0001 C CNN "MFP"
 	1    3200 4900
 	-1   0    0    1
@@
 P 4200 4600
 F 0 "D3" H 4200 4700 40  0000 C CNN
-F 1 "1n914" H 4200 4500 40  0000 C CNN
+F 1 "1n4148" H 4200 4500 40  0000 C CNN
 F 2 "Diodes_SMD:SOD-123" H 4200 4600 60  0001 C CNN
 F 3 "" H 4200 4600 60  0000 C CNN
+F 4 "1n4148W" H 4200 4600 60  0001 C CNN "MFN"
+F 5 "Vishay" H 4200 4600 60  0001 C CNN "MFP"
 	1    4200 4600
 	1    0    0    -1
@@
 P 4200 4900
 F 0 "D4" H 4200 5000 40  0000 C CNN
-F 1 "1n914" H 4200 4800 40  0000 C CNN
+F 1 "1n4148" H 4200 4800 40  0000 C CNN
 F 2 "Diodes_SMD:SOD-123" H 4200 4900 60  0001 C CNN
 F 3 "" H 4200 4900 60  0000 C CNN
+F 4 "1n4148W" H 4200 4900 60  0001 C CNN "MFN"
+F 5 "Vishay" H 4200 4900 60  0001 C CNN "MFP"
 	1    4200 4900
 	-1   0    0    1
@@
 F 2 "Capacitors_SMD:c_elec_5x5.8" H 6450 6700 60  0001 C CNN
 F 3 "" H 6450 6700 60  0000 C CNN
+F 4 "AVES106M35C12T-F" H 6450 6700 60  0001 C CNN "MFN"
+F 5 "Dubilier" H 6450 6700 60  0001 C CNN "MFP"
 	1    6450 6700
 	-1   0    0    -1
@@
 P 4400 6450
 F 0 "P1" H 4480 6450 40  0000 L CNN
-F 1 "CONN_1" H 4400 6505 30  0001 C CNN
+F 1 "NF" H 4400 6505 30  0001 C CNN
 F 2 "Socket_Strips:Socket_Strip_Straight_1x01" H 4400 6450 60  0001 C CNN
 F 3 "" H 4400 6450 60  0000 C CNN
+F 4 "~" H 4400 6450 60  0001 C CNN "MFN"
+F 5 "~" H 4400 6450 60  0001 C CNN "MFP"
 	1    4400 6450
 	-1   0    0    1
@@
 P 10325 3920
 F 0 "K4" V 10275 3920 50  0000 C CNN
-F 1 "CONN_3" V 10375 3920 40  0000 C CNN
+F 1 "NF" V 10375 3920 40  0000 C CNN
 F 2 "Socket_Strips:Socket_Strip_Straight_1x03" H 10325 3920 60  0001 C CNN
 F 3 "" H 10325 3920 60  0000 C CNN
@@
 P 5400 2700
 F 0 "K3" V 5350 2700 50  0000 C CNN
-F 1 "CONN_3" V 5450 2700 40  0000 C CNN
+F 1 "NF" V 5450 2700 40  0000 C CNN
 F 2 "Socket_Strips:Socket_Strip_Straight_1x03" H 5400 2700 60  0001 C CNN
 F 3 "" H 5400 2700 60  0000 C CNN
@@
 F 2 "Capacitors_SMD:c_elec_5x5.8" H 7665 4175 60  0001 C CNN
 F 3 "" H 7665 4175 60  0000 C CNN
+F 4 "AVES106M35C12T-F" H 7665 4175 60  0001 C CNN "MFN"
+F 5 "Dubilier" H 7665 4175 60  0001 C CNN "MFP"
 	1    7665 4175
 	-1   0    0    -1
@@
 P 6650 7050
 F 0 "P4" H 6730 7050 40  0000 L CNN
-F 1 "CONN_1" H 6650 7105 30  0001 C CNN
+F 1 "NF" H 6650 7105 30  0001 C CNN
 F 2 "Socket_Strips:Socket_Strip_Straight_1x01" H 6650 7050 60  0001 C CNN
 F 3 "" H 6650 7050 60  0000 C CNN
@@
 P 6850 7050
 F 0 "P5" H 6930 7050 40  0000 L CNN
-F 1 "CONN_1" H 6850 7105 30  0001 C CNN
+F 1 "NF" H 6850 7105 30  0001 C CNN
 F 2 "Socket_Strips:Socket_Strip_Straight_1x01" H 6850 7050 60  0001 C CNN
 F 3 "" H 6850 7050 60  0000 C CNN
+F 4 "~" H 6850 7050 60  0001 C CNN "MFN"
+F 5 "~" H 6850 7050 60  0001 C CNN "MFP"
 	1    6850 7050
 	0    -1   -1   0
@@
 F 2 "Socket_Strips:Socket_Strip_Straight_2x01" H 1650 4550 60  0001 C CNN
 F 3 "" H 1650 4550 60  0000 C CNN
+F 4 "640455-2" H 1650 4550 60  0001 C CNN "MFN"
+F 5 "TE Connectivity" H 1650 4550 60  0001 C CNN "MFP"
 	1    1650 4550
 	-1   0    0    1
@@
 P 4400 7200
 F 0 "P2" H 4480 7200 40  0000 L CNN
-F 1 "CONN_1" H 4400 7255 30  0001 C CNN
+F 1 "NF" H 4400 7255 30  0001 C CNN
 F 2 "Socket_Strips:Socket_Strip_Straight_1x01" H 4400 7200 60  0001 C CNN
 F 3 "" H 4400 7200 60  0000 C CNN
+F 4 "~" H 4400 7200 60  0001 C CNN "MFN"
+F 5 "~" H 4400 7200 60  0001 C CNN "MFP"
 	1    4400 7200
 	-1   0    0    1
@@
 F 2 "Housings_SSOP:MSOP-10_3x3mm_Pitch0.5mm" H 8330 3820 60  0001 C CNN
 F 3 "" H 8330 3820 60  0000 C CNN
+F 4 "ADS1115IDGST" H 8330 3820 60  0001 C CNN "MFN"
+F 5 "TI" H 8330 3820 60  0001 C CNN "MFP"
 	1    8330 3820
 	1    0    0    -1
@@
 P 8410 4750
 F 0 "L2" H 8410 4850 50  0000 C CNN
-F 1 "FERRITE BEAD" H 8410 4700 50  0000 C CNN
+F 1 "FERRITE BEAD" H 8780 4415 50  0000 C CNN
 F 2 "Choke_SMD:Choke_SMD_1206_Standard" H 8410 4750 60  0001 C CNN
 F 3 "" H 8410 4750 60  0000 C CNN
+F 4 "2512061217Y5" H 8410 4750 60  0001 C CNN "MFN"
+F 5 "Fair-rite" H 8410 4750 60  0001 C CNN "MFP"
 	1    8410 4750
 	0    -1   -1   0
@@
 	8410 5000 8410 5545
 Wire Wire Line
-	7665 3000 7660 3000
+	7230 3000 7665 3000
 Connection ~ 7660 3000
 Wire Wire Line
 	8410 3010 8410 3005
 Wire Wire Line
-	7665 4085 7665 3000
+	7665 3000 7665 4085
 $Comp
 L INDUCTOR_SMALL L1
@@
 F 2 "Choke_SMD:Choke_SMD_1206_Standard" H 6980 3000 60  0001 C CNN
 F 3 "" H 6980 3000 60  0000 C CNN
+F 4 "2512061217Y5" H 6980 3000 60  0001 C CNN "MFN"
+F 5 "Fair-rite" H 6980 3000 60  0001 C CNN "MFP"
 	1    6980 3000
 	1    0    0    -1
@@
 	6200 3000 6730 3000
 Wire Wire Line
-	7230 3000 8410 3000
+	7660 3000 8410 3000
 $Comp
 L 11aa02e48 U2
@@
 F 2 "Housings_SOT-23_SOT-143_TSOT-6:SOT-23" H 9255 1595 60  0001 C CNN
 F 3 "" H 9255 1595 60  0000 C CNN
+F 4 "11aa02e48-I/TT" H 9255 1595 60  0001 C CNN "MFN"
+F 5 "Microchip" H 9255 1595 60  0001 C CNN "MFP"
 	1    9255 1595
 	1    0    0    -1
